File: kicad/AudioBalancer.kicad_pcb (KiCad board)
At the start: 2 copper layers, 47 x 65.4 mm, 41 parts, among them J1 Conn_01x03_Pin, J2 Conn_01x02_Pin, J3 Conn_01x02_Pin, J4 Conn_01x03_Pin, J5 Conn_01x03_Pin, U1 SSM2141, U2 SSM2142P

Commit message: Changed to protection values in 'The 48 Volt Phantom Menace Returns'
Parts:
- D1, D2, D3, D4, D5, D6, D7, D8: value SB160 -> 1N4004GP
- R2, R3: value 4R9 -> 47R
